File: clock_pcb/PAGE2.kicad_sch (KiCad schematic)
At the start: 69 parts, among them J1 USB_C_Receptacle_USB2.0, J2 PROG, Q1 AO3401A, Q2 AO3401A, SW1 TS-1187A-B-A-B, SW2 SSSS811101, SW3 TS-1187A-B-A-B, U1 SRV05-4, U2 RP2040, U3 RT9080-33GJ5, U4 W25Q64JV, Y1 XYDBPCNANF-12MHZ

Commit message: break
Parts:
- removed C5: 0.1u, Capacitor_SMD:C_0402_1005Metric, symbol Device:C_Small
- D1: value IO -> LED; Color (none) -> YLW; desc Yellow -> VFtyp 2V, VFmax 2.3V, Yellow
- D3: value 5V Blue -> LED; Color (none) -> BLU; desc (none) -> VFtyp 2.8V, VFmax 3.1V, Blue
- D4: value 3V3 Blue -> LED; Color (none) -> GRN; desc (none) -> VFtyp 3.3V, VFmax 3.7V, Green; lcsc C72041 -> C72043
- H4, H5, H6, H7: footprint MountingHole:MountingHole_3.2mm_M3 -> MountingHole:MountingHole_2.7mm_M2.5
- TP1: value 5V -> VBUS
- TP2: value 5V -> GND
- TP3: value 5V -> RST
- TP6: value 5V -> 3V3
- renumbered C11 to C10, C12 to C11, C13 to C12, C14 to C13, C15 to C14, C16 to C15, C17 to C16, C18 to C17, C19 to C18, C6 to C5, C7 to C6, C8 to C7, C9 to C8, C10 to C9, R4 to R3, R5 to R4, R3 to R5
Connections:
- net +3V3: no longer R5.2
- net GND: now also D1.1 (K)
- net USB_D+: now also U1.3 (IO2); no longer U1.1 (IO1)
- net USB_D-: now also U1.1 (IO1); no longer U1.3 (IO2)
- net PWR_OFF_SW_N: now reaches R8.2, R9.2, SW2.3 (C)
- net GPIO12 renamed GPIO12_PPS
- net GPIO13 renamed GPIO13_WS2812_RGB_LED
- net GPIO14 renamed GPIO14_BUTTON_0
- net GPIO15 renamed GPIO15_BUTTON_1
- net GPIO25 renamed GPIO25_LED
- net GPIO25_LED: now also R5.2; no longer D1.1 (K)
- net GPIO26 renamed GPIO26_ADC0_LDR
- net GPIO27 renamed GPIO27_ADC1
- net GPIO28 renamed GPIO28_ADC2
- net GPIO29 renamed GPIO29_ADC3
- net I2C0_SCL renamed I2C_SCL
- net I2C0_SDA renamed I2C_SDA
- no-connect marks 8 -> 14
Other:
- note added: "ADC4 Connected to internal temp sense"
- note removed: "--->USER LED"
- note removed: "ADC"
- moved on the sheet: C1, C10, C11, C12, C13, C14, C15, C18, C2, C3, C4, C5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

Commit message: only brick nogging usbc left to add
Parts:
- added TP8: GND CLIP, Mitch_Library:ronghe_RH-5016_C5199799, symbol Connector:TestPoint
Connections:
- net GND: now also TP8.1
- no-connect marks 14 -> 5
Other:
- moved on the sheet: C1, C10, C11, C12, C13, C14, C15, C18, C2, C3, C4, C5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
